File: PCB-Keyboard-EDIPO.kicad_pcb (KiCad board)
At the start: 2 copper layers, 155 parts, among them J1 AVR-ISP-6, SW1 ESC`, SW10 #9, SW11 #0, SW12 -_, SW13 =+, SW14 BACKSPACE, SW15 DELETE, SW16 TAB, SW17 Q, SW18 W, SW19 E, SW2 #1, SW20 R, SW21 T, SW22 Y, SW23 U, SW24 I, SW25 O, SW26 P, SW27 [{, SW28 }], SW29 \|, SW3 #2, SW30 F1, SW31 CAPSLOCK, SW32 A, SW33 S, SW34 D, SW35 F, SW36 G, SW37 H, SW38 J, SW39 K, SW4 #3, SW40 L, SW41 ;:, SW42 '", SW43 ENTER, SW44 F2, SW45 SHIFT, SW46 Z, SW47 X, SW48 C, SW49 V, SW5 #4, SW50 B, SW51 N, SW52 M, SW53 ,<, SW54 .>, SW55 /?, SW56 FN, SW57 UP, SW58 F3, SW59 CTRL, SW6 #5, SW60 ALT, SW61 COMMAND, SW62 SPACE, SW63 ALT, SW64 `~, SW65 LEFT, SW66 DOWN, SW67 RIGHT, SW68 SW_Push_Reset, SW7 #6, SW8 #7, SW9 #8, U1 ATmega32U4-A, U2 PRTR5V0U2X, Y1 XTAL

Commit message: Alight PCB Matrix
Parts:
- C1, C2, C3, C4, C5, C6, C7, C8, D1, D10, D11, D12, D13, D14, D15, D16, D17, D18, D19, D2, D20, D21, D22, D23, D24, D25, D26, D27, D28, D29, D3, D30, D31, D32, D33, D34, D35, D36, D37, D38, D39, D4, D40, D41, D42, D43, D44, D45, D46, D47, D48, D49, D5, D50, D51, D52, D53, D54, D55, D56, D57, D58, D59, D6, D60, D61, D62, D63, D64, D65, D66, D67, D7, D8, D9, F1, J1, R1, R2, R3, R4, R5, R6, SW68, U1, U2, USB1, Y1: moved to B.Cu
- moved SW30 353.7 mm to (331.1, -161.9)
- moved SW15 347.4 mm to (331.1, -180.9)
- moved SW29 333.6 mm to (307.3, -161.9)
- moved SW14 323.6 mm to (302.5, -180.9)
- moved SW10 318.9 mm to (216.8, -180.9)
- moved SW28 314.2 mm to (283.5, -161.9)
- moved SW9 305.4 mm to (197.8, -180.9)
- moved SW13 300.9 mm to (274.0, -180.9)
- moved SW58 298.2 mm to (331.1, -123.8)
- moved SW27 298.0 mm to (264.4, -161.9)
- moved SW44 297.6 mm to (331.1, -142.8)
- moved SW8 292.7 mm to (178.7, -180.9)
- moved SW12 284.4 mm to (254.9, -180.9)
- moved SW26 282.4 mm to (245.4, -161.9)
- moved SW7 280.9 mm to (159.7, -180.9)
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
Commit message: Switch (SW_PUSH) Orientation Flip
rotated SW_PUSH in schematic to align with tutorial
Parts:
- moved C3 349.5 mm to (259.3, -132.0)
- moved C4 349.5 mm to (259.3, -129.0)
- moved C6 349.5 mm to (259.3, -123.0)
- moved C7 349.5 mm to (259.3, -120.0)
- moved R3 349.5 mm to (254.6, -132.2)
- moved R4 349.5 mm to (254.6, -129.2)
- moved R5 349.5 mm to (254.6, -126.3)
- moved C2 349.5 mm to (259.3, -135.0)
- moved C5 349.5 mm to (259.3, -126.0)
- moved C8 349.5 mm to (259.3, -117.0)
- moved R2 349.5 mm to (254.6, -135.1)
- moved R6 349.5 mm to (254.6, -123.3)
- moved U2 349.5 mm to (254.9, -119.8)
- moved C1 341.9 mm to (272.8, -132.8)
- moved F1 341.9 mm to (226.7, -113.8)
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Connections:
- SW1 pad 1: Net-(D1-A) -> col0
- SW1 pad 2: col0 -> Net-(D1-A)
- SW10 pad 1: Net-(D10-A) -> col9
- SW10 pad 2: col9 -> Net-(D10-A)
- SW11 pad 1: Net-(D11-A) -> col10
- SW11 pad 2: col10 -> Net-(D11-A)
- SW12 pad 1: Net-(D12-A) -> col11
- SW12 pad 2: col11 -> Net-(D12-A)
- SW13 pad 1: Net-(D13-A) -> col12
- SW13 pad 2: col12 -> Net-(D13-A)
- SW14 pad 1: Net-(D14-A) -> col13
- SW14 pad 2: col13 -> Net-(D14-A)
- SW15 pad 1: Net-(D15-A) -> col14
- SW15 pad 2: col14 -> Net-(D15-A)
- SW16 pad 1: Net-(D16-A) -> col0
- SW16 pad 2: col0 -> Net-(D16-A)
- SW17 pad 1: Net-(D17-A) -> col1
- SW17 pad 2: col1 -> Net-(D17-A)
- SW18 pad 1: Net-(D18-A) -> col2
- SW18 pad 2: col2 -> Net-(D18-A)
- SW19 pad 1: Net-(D19-A) -> col3
- SW19 pad 2: col3 -> Net-(D19-A)
- SW2 pad 1: Net-(D2-A) -> col1
- SW2 pad 2: col1 -> Net-(D2-A)
- SW20 pad 1: Net-(D20-A) -> col4
- SW20 pad 2: col4 -> Net-(D20-A)
- SW21 pad 1: Net-(D21-A) -> col5
- SW21 pad 2: col5 -> Net-(D21-A)
- SW22 pad 1: Net-(D22-A) -> col6
- SW22 pad 2: col6 -> Net-(D22-A)
- SW23 pad 1: Net-(D23-A) -> col7
- SW23 pad 2: col7 -> Net-(D23-A)
- SW24 pad 1: Net-(D24-A) -> col8
- SW24 pad 2: col8 -> Net-(D24-A)
- SW25 pad 1: Net-(D25-A) -> col9
- SW25 pad 2: col9 -> Net-(D25-A)
- SW26 pad 1: Net-(D26-A) -> col10
- SW26 pad 2: col10 -> Net-(D26-A)
- SW27 pad 1: Net-(D27-A) -> col11
- SW27 pad 2: col11 -> Net-(D27-A)
- SW28 pad 1: Net-(D28-A) -> col12
- SW28 pad 2: col12 -> Net-(D28-A)
- SW29 pad 1: Net-(D29-A) -> col13
- SW29 pad 2: col13 -> Net-(D29-A)
- SW3 pad 1: Net-(D3-A) -> col2
- SW3 pad 2: col2 -> Net-(D3-A)
- SW30 pad 1: Net-(D30-A) -> col14
- SW30 pad 2: col14 -> Net-(D30-A)
- SW31 pad 1: Net-(D31-A) -> col0
- SW31 pad 2: col0 -> Net-(D31-A)
- SW32 pad 1: Net-(D32-A) -> col1
- SW32 pad 2: col1 -> Net-(D32-A)
- SW33 pad 1: Net-(D33-A) -> col2
- SW33 pad 2: col2 -> Net-(D33-A)
- SW34 pad 1: Net-(D34-A) -> col3
- SW34 pad 2: col3 -> Net-(D34-A)
- SW35 pad 1: Net-(D35-A) -> col4
- SW35 pad 2: col4 -> Net-(D35-A)
- SW36 pad 1: Net-(D36-A) -> col5
- SW36 pad 2: col5 -> Net-(D36-A)
- SW37 pad 1: Net-(D37-A) -> col6
- SW37 pad 2: col6 -> Net-(D37-A)
- SW38 pad 1: Net-(D38-A) -> col7
- SW38 pad 2: col7 -> Net-(D38-A)
- SW39 pad 1: Net-(D39-A) -> col8
- SW39 pad 2: col8 -> Net-(D39-A)
- SW4 pad 1: Net-(D4-A) -> col3
- SW4 pad 2: col3 -> Net-(D4-A)
- SW40 pad 1: Net-(D40-A) -> col9
- SW40 pad 2: col9 -> Net-(D40-A)
- SW41 pad 1: Net-(D41-A) -> col10
- SW41 pad 2: col10 -> Net-(D41-A)
- SW42 pad 1: Net-(D42-A) -> col11
- SW42 pad 2: col11 -> Net-(D42-A)
- SW43 pad 1: Net-(D43-A) -> col13
- SW43 pad 2: col13 -> Net-(D43-A)
- SW44 pad 1: Net-(D44-A) -> col14
- SW44 pad 2: col14 -> Net-(D44-A)
- SW45 pad 1: Net-(D45-A) -> col0
- SW45 pad 2: col0 -> Net-(D45-A)
- SW46 pad 1: Net-(D46-A) -> col1
- SW46 pad 2: col1 -> Net-(D46-A)
- SW47 pad 1: Net-(D47-A) -> col2
- SW47 pad 2: col2 -> Net-(D47-A)
- SW48 pad 1: Net-(D48-A) -> col3
- SW48 pad 2: col3 -> Net-(D48-A)
- SW49 pad 1: Net-(D49-A) -> col4
- SW49 pad 2: col4 -> Net-(D49-A)
- SW5 pad 1: Net-(D5-A) -> col4
- SW5 pad 2: col4 -> Net-(D5-A)
- SW50 pad 1: Net-(D50-A) -> col5
- SW50 pad 2: col5 -> Net-(D50-A)
- SW51 pad 1: Net-(D51-A) -> col6
- SW51 pad 2: col6 -> Net-(D51-A)
- SW52 pad 1: Net-(D52-A) -> col7
- SW52 pad 2: col7 -> Net-(D52-A)
- SW53 pad 1: Net-(D53-A) -> col8
- SW53 pad 2: col8 -> Net-(D53-A)
- SW54 pad 1: Net-(D54-A) -> col9
- SW54 pad 2: col9 -> Net-(D54-A)
- SW55 pad 1: Net-(D55-A) -> col10
- SW55 pad 2: col10 -> Net-(D55-A)
- SW56 pad 1: Net-(D56-A) -> col12
- SW56 pad 2: col12 -> Net-(D56-A)
- SW57 pad 1: Net-(D57-A) -> col13
- SW57 pad 2: col13 -> Net-(D57-A)
- SW58 pad 1: Net-(D58-A) -> col14
- SW58 pad 2: col14 -> Net-(D58-A)
- SW59 pad 1: Net-(D59-A) -> col0
- SW59 pad 2: col0 -> Net-(D59-A)
- SW6 pad 1: Net-(D6-A) -> col5
- SW6 pad 2: col5 -> Net-(D6-A)
- SW60 pad 1: Net-(D60-A) -> col1
- SW60 pad 2: col1 -> Net-(D60-A)
- SW61 pad 1: Net-(D61-A) -> col2
- SW61 pad 2: col2 -> Net-(D61-A)
- SW62 pad 1: Net-(D62-A) -> col6
- SW62 pad 2: col6 -> Net-(D62-A)
- SW63 pad 1: Net-(D63-A) -> col10
- SW63 pad 2: col10 -> Net-(D63-A)
- SW64 pad 1: Net-(D64-A) -> col11
- SW64 pad 2: col11 -> Net-(D64-A)
- SW65 pad 1: Net-(D65-A) -> col12
- SW65 pad 2: col12 -> Net-(D65-A)
- SW66 pad 1: Net-(D66-A) -> col13
- SW66 pad 2: col13 -> Net-(D66-A)
- SW67 pad 1: Net-(D67-A) -> col14
- SW67 pad 2: col14 -> Net-(D67-A)
- SW7 pad 1: Net-(D7-A) -> col6
- SW7 pad 2: col6 -> Net-(D7-A)
- SW8 pad 1: Net-(D8-A) -> col7
- SW8 pad 2: col7 -> Net-(D8-A)
- SW9 pad 1: Net-(D9-A) -> col8
- SW9 pad 2: col8 -> Net-(D9-A)

Commit message: PCB Component Movement 1
Parts:
- moved D1 172.5 mm to (21.8, -141.0), turned to 90 degrees
- moved D16 162.9 mm to (26.3, -121.9), turned to 90 degrees
- moved D31 156.0 mm to (28.6, -102.9), turned to 90 degrees
- moved D67 155.2 mm to (307.0, -64.8), turned to 90 degrees
- moved D2 153.3 mm to (40.9, -141.1), turned to 90 degrees
- moved D59 153.3 mm to (26.0, -64.8), turned to 90 degrees
- moved D45 148.1 mm to (33.5, -83.8), turned to 90 degrees
- moved D58 140.2 mm to (307.0, -83.8), turned to 90 degrees
- moved D66 139.7 mm to (288.0, -64.8), turned to 90 degrees
- moved D17 138.9 mm to (50.0, -122.0), turned to 90 degrees
- moved D3 134.5 mm to (59.7, -140.8), turned to 90 degrees
- moved D44 131.9 mm to (307.0, -103.1), turned to 90 degrees
- moved D32 129.8 mm to (54.6, -102.9), turned to 90 degrees
- moved D60 127.3 mm to (52.5, -64.8), turned to 90 degrees
- moved R1 125.8 mm to (187.2, -36.4)
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Connections:
- F1 pad 1: VCC -> +5V
- F1 pad 2: +5V -> VCC
- R2 pad 1: Reset -> RESET
- R5 pad 1: GND -> Net-(USB1-CC2)
- R5 pad 2: Net-(USB1-CC2) -> GND
- R6 pad 1: GND -> Net-(USB1-CC1)
- R6 pad 2: Net-(USB1-CC1) -> GND
- SW68 pad 1: Reset -> RESET
