File: PCB-Keyboard-EDIPO.kicad_pcb (KiCad board)
At the start: 2 copper layers, 304.8 x 99.8 mm, 155 parts, among them J1 AVR-ISP-6, SW1 ESC`, SW10 #9, SW11 #0, SW12 -_, SW13 =+, SW14 BACKSPACE, SW15 DELETE, SW16 TAB, SW17 Q, SW18 W, SW19 E, SW2 #1, SW20 R, SW21 T, SW22 Y, SW23 U, SW24 I, SW25 O, SW26 P, SW27 [{, SW28 }], SW29 \|, SW3 #2, SW30 F1, SW31 CAPSLOCK, SW32 A, SW33 S, SW34 D, SW35 F, SW36 G, SW37 H, SW38 J, SW39 K, SW4 #3, SW40 L, SW41 ;:, SW42 '", SW43 ENTER, SW44 F2, SW45 SHIFT, SW46 Z, SW47 X, SW48 C, SW49 V, SW5 #4, SW50 B, SW51 N, SW52 M, SW53 ,<, SW54 .>, SW55 /?, SW56 FN, SW57 UP, SW58 F3, SW59 CTRL, SW6 #5, SW60 ALT, SW61 COMMAND, SW62 SPACE, SW63 ALT, SW64 `~, SW65 LEFT, SW66 DOWN, SW67 RIGHT, SW68 SW_Push_Reset, SW7 #6, SW8 #7, SW9 #8, U1 ATmega32U4-A, U2 PRTR5V0U2X, Y1 XTAL

Commit message: Wires
Routing:
- net col14: track 0.00 -> 133.3 mm
- net col1: track 0.00 -> 91.0 mm
- net col10: track 0.00 -> 89.0 mm
- net col6: track 0.00 -> 88.0 mm
- net col2: track 0.00 -> 88.0 mm
- net col13: track 0.00 -> 86.1 mm
- net col12: track 0.00 -> 84.1 mm
- net col0: track 0.00 -> 84.1 mm
- net col11: track 0.00 -> 84.1 mm
- net DN: track 0.00 -> 77.8 mm
- net DP: track 0.00 -> 75.9 mm
- net col4: track 0.00 -> 67.1 mm
- net col9: track 0.00 -> 67.0 mm
- net col7: track 0.00 -> 67.0 mm
- net col8: track 0.00 -> 67.0 mm
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
Commit message: Routing 1
Parts:
- moved R4 4.78 mm to (179.8, -81.7)
- moved R3 4.78 mm to (177.7, -81.7)
- moved C1 4.23 mm to (183.6, -77.0)
- moved C6 3.64 mm to (196.6, -71.4), turned to 0 degrees
- moved C3 3.60 mm to (202.7, -64.3)
- moved C2 3.30 mm to (202.7, -67.5)
- moved C8 1.80 mm to (178.7, -74.6), turned to 135 degrees
- moved C4 1.68 mm to (190.3, -57.2)
- moved R1 1.16 mm to (177.0, -57.2)
- moved C7 0.78 mm to (174.4, -69.8), turned to 180 degrees
- moved D39 0.51 mm to (198.5, -99.4)
- moved D40 0.51 mm to (217.5, -99.4)
- moved D3 0.51 mm to (70.2, -137.5)
- moved D4 0.51 mm to (89.1, -137.5)
- moved C5 0.46 mm to (174.9, -61.9), turned to 180 degrees
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Routing:
- net row0: track 0.00 -> 304.7 mm, vias 0 -> 2
- net row2: track 0.00 -> 295.3 mm, vias 0 -> 2
- net row1: track 0.00 -> 278.2 mm
- net row3: track 0.00 -> 268.5 mm
- net row4: track 0.00 -> 214.4 mm
- net GND: track 0.00 -> 207.1 mm, vias 0 -> 8
- net +5V: track 0.00 -> 156.1 mm, vias 0 -> 6
- net VCC: track 0.00 -> 23.4 mm, vias 0 -> 2
- net XTAL1: track 0.00 -> 14.6 mm
- net XTAL2: track 0.00 -> 13.8 mm
- net Net-(D8-A): track 0.00 -> 9.43 mm
- net Net-(D9-A): track 0.00 -> 6.58 mm
- net Net-(D60-A): track 0.00 -> 6.52 mm
- net Net-(D61-A): track 0.00 -> 6.50 mm
- net Net-(D45-A): track 0.00 -> 6.44 mm
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- added copper zone on B.Cu, net (none)
- added copper zone on F.Cu, net (none)

Commit message: Rough Routing Completed
Must now fix errors if any
Parts:
- moved J1 70.5 mm to (214.8, -70.9)
- moved R2 10.6 mm to (209.0, -61.0)
- moved SW68 2.25 mm to (215.2, -63.0), turned to 0 degrees
- moved R1 1.68 mm to (178.5, -58.0)
- moved C4 0.89 mm to (189.7, -57.9)
- moved C5 0.49 mm to (174.4, -61.9)
Connections:
- U1 pad 1: row0 -> row3
- U1 pad 22: col12 -> col11
- U1 pad 25: col11 -> col12
- U1 pad 36: col4 -> row4
- U1 pad 38: row1 -> col6
- U1 pad 39: row4 -> row0
- U1 pad 40: row3 -> row1
Routing:
- net row0: track 304.7 -> 511.3 mm
- net row1: track 278.2 -> 464.4 mm
- net col0: track 84.1 -> 251.8 mm, vias 0 -> 1
- net row2: track 295.3 -> 461.0 mm
- net col1: track 91.0 -> 231.6 mm, vias 0 -> 1
- net col14: track 133.3 -> 272.9 mm, vias 0 -> 1
- net col13: track 86.1 -> 205.6 mm, vias 0 -> 1
- net col2: track 88.0 -> 201.1 mm, vias 0 -> 1
- net col3: track 67.0 -> 172.2 mm, vias 0 -> 1
- net col12: track 84.1 -> 183.2 mm, vias 0 -> 1
- net row4: track 214.4 -> 308.8 mm, vias 0 -> 2
- net col4: track 67.1 -> 152.2 mm, vias 0 -> 1
- net col11: track 84.1 -> 158.6 mm, vias 0 -> 1
- net col9: track 67.0 -> 126.7 mm, vias 0 -> 1
- net col10: track 89.0 -> 141.4 mm, vias 0 -> 1
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