File: PCB-Keyboard-EDIPO.kicad_pcb (KiCad board)
At the start: 2 copper layers, 304.8 x 99.8 mm, 155 parts, among them J1 AVR-ISP-6, SW1 ESC`, SW10 #9, SW11 #0, SW12 -_, SW13 =+, SW14 BACKSPACE, SW15 DELETE, SW16 TAB, SW17 Q, SW18 W, SW19 E, SW2 #1, SW20 R, SW21 T, SW22 Y, SW23 U, SW24 I, SW25 O, SW26 P, SW27 [{, SW28 }], SW29 \|, SW3 #2, SW30 F1, SW31 CAPSLOCK, SW32 A, SW33 S, SW34 D, SW35 F, SW36 G, SW37 H, SW38 J, SW39 K, SW4 #3, SW40 L, SW41 ;:, SW42 '", SW43 ENTER, SW44 F2, SW45 SHIFT, SW46 Z, SW47 X, SW48 C, SW49 V, SW5 #4, SW50 B, SW51 N, SW52 M, SW53 ,<, SW54 .>, SW55 /?, SW56 FN, SW57 UP, SW58 F3, SW59 CTRL, SW6 #5, SW60 ALT, SW61 COMMAND, SW62 SPACE, SW63 ALT, SW64 `~, SW65 LEFT, SW66 DOWN, SW67 RIGHT, SW68 SW_Push_Reset, SW7 #6, SW8 #7, SW9 #8, U1 ATmega32U4-A, U2 PRTR5V0U2X, Y1 XTAL

Commit message: Logo
Parts:
- added G***: LOGO, Alps_Only:EdipoSLogo, F.Cu at (125.4, -65.9)
- added G***: LOGO, Alps_Only:EdipoSLogo, B.Cu at (125.4, -65.9)
Routing:
- net (no net): track 0.00 -> 15.0 mm, vias 0 -> 12
Other:
- board size 304.8 x 99.8 mm -> 304.8 x 100.8 mm
- board text added: "v1.0.0 - © Edipo 2025"

Commit message: Via Stitching to ground
Routing:
- net GND: track 279.9 -> 325.9 mm, vias 9 -> 106
- net (no net): track 15.0 -> 0.00 mm, vias 12 -> 0
- net DP: track 75.2 -> 74.5 mm
- net DN: track 72.9 -> 72.1 mm
- added copper zone on B.Cu, net GND
- added copper zone on F.Cu, net GND
- removed copper zone on B.Cu, net (none)
- removed copper zone on F.Cu, net (none)

Commit message: PCB v1.0.1
Parts:
- added FB1: 60@100MHz, Inductor_SMD:L_0805_2012Metric_Pad1.15x1.40mm_HandSolder, B.Cu at (178.6, -147.2)
Connections:
- USB1 pad 13: GND -> Earth
Routing:
- net Earth: track 0.00 -> 23.4 mm, vias 0 -> 5
- net GND: track 325.9 -> 304.8 mm, vias 106 -> 114
- added copper zone on B.Cu, net Earth
- added copper zone on F.Cu, net Earth
