File: PCB-Keyboard-EDIPO-ALPS.kicad_pcb (KiCad board)
At the start: 2 copper layers, 304.8 x 100.8 mm, 158 parts, among them J1 AVR-ISP-6, SW1 ESC`, SW10 #9, SW11 #0, SW12 -_, SW13 =+, SW14 BACKSPACE, SW15 DELETE, SW16 TAB, SW17 Q, SW18 W, SW19 E, SW2 #1, SW20 R, SW21 T, SW22 Y, SW23 U, SW24 I, SW25 O, SW26 P, SW27 [{, SW28 }], SW29 \|, SW3 #2, SW30 F1, SW31 CAPSLOCK, SW32 A, SW33 S, SW34 D, SW35 F, SW36 G, SW37 H, SW38 J, SW39 K, SW4 #3, SW40 L, SW41 ;:, SW42 '", SW43 ENTER, SW44 F2, SW45 SHIFT, SW46 Z, SW47 X, SW48 C, SW49 V, SW5 #4, SW50 B, SW51 N, SW52 M, SW53 ,<, SW54 .>, SW55 /?, SW56 FN, SW57 UP, SW58 F3, SW59 CTRL, SW6 #5, SW60 ALT, SW61 COMMAND, SW62 SPACE, SW63 ALT, SW64 `~, SW65 LEFT, SW66 DOWN, SW67 RIGHT, SW68 SW_Push_Reset, SW7 #6, SW8 #7, SW9 #8, U1 ATmega32U4-A, U2 PRTR5V0U2X, Y1 XTAL

Commit message: zoning
Routing:
- net (no net): track 0.00 -> 2.38 mm
Changed lines of the file:
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@@
+	)
+	(segment
+		(start 177.8 -138.1125)
+		(end 177.8 -137.31875)
+		(width 0.2)
+		(layer "B.Cu")
+		(net 0)
+	)
+	(segment
+		(start 177.8 -137.31875)
+		(end 177.8 -138.90625)
+		(width 0.2)
+		(layer "B.Cu")
+		(net 0)
 	)
 	(segment
