File: PCB-Keyboard-EDIPO-ALPS.kicad_pcb (KiCad board)
At the start: 2 copper layers, 304.8 x 100.8 mm, 158 parts, among them J1 AVR-ISP-6, SW1 ESC`, SW10 #9, SW11 #0, SW12 -_, SW13 =+, SW14 BACKSPACE, SW15 DELETE, SW16 TAB, SW17 Q, SW18 W, SW19 E, SW2 #1, SW20 R, SW21 T, SW22 Y, SW23 U, SW24 I, SW25 O, SW26 P, SW27 [{, SW28 }], SW29 \|, SW3 #2, SW30 F1, SW31 CAPSLOCK, SW32 A, SW33 S, SW34 D, SW35 F, SW36 G, SW37 H, SW38 J, SW39 K, SW4 #3, SW40 L, SW41 ;:, SW42 '", SW43 ENTER, SW44 F2, SW45 SHIFT, SW46 Z, SW47 X, SW48 C, SW49 V, SW5 #4, SW50 B, SW51 N, SW52 M, SW53 ,<, SW54 .>, SW55 /?, SW56 FN, SW57 UP, SW58 F3, SW59 CTRL, SW6 #5, SW60 ALT, SW61 COMMAND, SW62 SPACE, SW63 ALT, SW64 `~, SW65 LEFT, SW66 DOWN, SW67 RIGHT, SW68 SW_Push_Reset, SW7 #6, SW8 #7, SW9 #8, U1 ATmega32U4-A, U2 PRTR5V0U2X, Y1 XTAL

Commit message: usb
Routing:
- net col14: track 216.0 -> 214.8 mm
- net Earth: track 23.4 -> 24.3 mm
- net GND: vias 113 -> 115
Other:
- board size 304.8 x 100.8 mm -> 304.8 x 99.8 mm

Commit message: Finished PCB
Parts:
- SW60: footprint Alps_Only:ALPS-1.25U -> MX_Only:MXOnly-1.25U-NoLED
- moved D11 218.4 mm to (266.1, 77.3)
- moved D12 218.4 mm to (285.0, 77.3)
- moved SW13 218.4 mm to (296.3, 74.8)
- moved SW41 218.4 mm to (272.5, 112.9)
- moved SW64 218.4 mm to (296.3, 151.0)
- moved C1 218.4 mm to (224.7, 139.4)
- moved C2 218.4 mm to (243.4, 147.1)
- moved C3 218.4 mm to (243.4, 150.2)
- moved C4 218.4 mm to (230.4, 156.6)
- moved C5 218.4 mm to (215.1, 152.6)
- moved C6 218.4 mm to (237.3, 143.1)
- moved C7 218.4 mm to (215.1, 144.7)
- moved C8 218.4 mm to (219.4, 140.0)
- moved D1 218.4 mm to (76.0, 77.0)
- moved D10 218.4 mm to (247.0, 77.3)
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Routing:
- net col1: track 228.3 -> 233.1 mm
- net Net-(D60-A): track 9.42 -> 10.0 mm
Other:
- board text added: "#0"
- board text added: "#1"
- board text added: "#9"
- board text added: "'{dblquote}"
- board text added: ",<"
- board text added: "-_"
- board text added: ".>"
- board text added: "/?"
- board text added: ";:"
- board text added: "=+"
- board text added: "A"
- board text added: "ALT"
- board text added: "BACKSPACE"
- board text added: "CAPSLOCK"
- board text added: "COMMAND"
- board text added: "CTRL"
- board text added: "DELETE"
- board text added: "DOWN"
- board text added: "ENTER"
- board text added: "ESC"
- board text added: "F1"
- board text added: "F2"
- board text added: "F3"
- board text added: "FN"
- board text added: "L"
- board text added: "LEFT"
- board text added: "M"
- board text added: "P"
- board text added: "Q"
- board text added: "RIGHT"
- board text added: "SHIFT"
- board text added: "SPACE"
- board text added: "TAB"
- board text added: "UP"
- board text added: "Z"
- board text added: "[{"
- board text added: "\|"
- board text added: "]}"
- board text added: "`~"

Commit message: Fixed Last Traces
Routing:
- net col1: track 233.1 -> 229.4 mm
Other:
- board text removed: "#0"
- board text removed: "#1"
- board text removed: "#9"
- board text removed: "'{dblquote}"
- board text removed: ",<"
- board text removed: "-_"
- board text removed: ".>"
- board text removed: "/?"
- board text removed: ";:"
- board text removed: "=+"
- board text removed: "A"
- board text removed: "ALT"
- board text removed: "BACKSPACE"
- board text removed: "CAPSLOCK"
- board text removed: "COMMAND"
- board text removed: "CTRL"
- board text removed: "DELETE"
- board text removed: "DOWN"
- board text removed: "ENTER"
- board text removed: "ESC"
- board text removed: "F1"
- board text removed: "F2"
- board text removed: "F3"
- board text removed: "FN"
- board text removed: "L"
- board text removed: "LEFT"
- board text removed: "M"
- board text removed: "P"
- board text removed: "Q"
- board text removed: "RIGHT"
- board text removed: "SHIFT"
- board text removed: "SPACE"
- board text removed: "TAB"
- board text removed: "UP"
- board text removed: "Z"
- board text removed: "[{"
- board text removed: "\|"
- board text removed: "]}"
- board text removed: "`~"
