File: _autosave-PCB-Keyboard-EDIPO.kicad_sch (KiCad schematic)
At the start: 21 parts, among them J1 AVR-ISP-6, SW68 SW_Push_Reset, U1 ATmega32U4-A, U2 PRTR5V0U2X, Y1 XTAL

Commit message: zoning
Parts:
- added FB1: 60@100MHz, Inductor_SMD:L_0805_2012Metric_Pad1.15x1.40mm_HandSolder, symbol Device:FerriteBead_Small
Connections:
- net GND: now also FB1.2; no longer USB1.13 (SHIELD)
- new net Earth: FB1.1, USB1.13 (SHIELD)
Other:
- moved on the sheet: J1
