File: PCB-Keyboard-EDIPO.kicad_sch (KiCad schematic)
At the start: 30 parts, among them J1 USB_C_Receptacle_USB2.0_16P, J2 Conn_01x04, J3 Conn_01x05, SW1 SW_Push, SW2 SW_Push, U1 RP2040, U2 XC6206PxxxMR, U3 W25Q128JVS, U4 SRV05-4, Y1 Crystal_GND24

Commit message: new schema
Parts:
- added R5, R6: 5.1k, symbol Device:R_Small
Connections:
- net +3V3: now also R6.2
- net Q_SEL: now also R5.1
- new net: R5.2, R6.1
Other:
- moved on the sheet: R4, SW2

Commit message: pcb keyboard 2
Parts:
- added C1, C10, C11, C12, C13, C14, C15, C16, C17, C18, C19, C2, C20, C21, C22, C23, C24, C25, C26, C27, C28, C29, C3, C30, C31, C32, C33, C34, C35, C36, C37, C38, C39, C4, C40, C41, C42, C43, C44, C45, C46, C47, C48, C49, C5, C50, C51, C52, C53, C54, C55, C56, C57, C58, C59, C6, C60, C61, C62, C63, C64, C65, C66, C67, C68, C69, C7, C70, C71, C72, C73, C74, C75, C76, C77, C78, C79, C8, C9, C92, C93, C94, C95: 100n, Capacitor_SMD:C_0805_2012Metric_Pad1.18x1.45mm_HandSolder, symbol Device:C_Small
- added D1, D10, D11, D12, D13, D14, D15, D16, D17, D18, D19, D2, D20, D21, D22, D23, D24, D25, D26, D27, D28, D29, D3, D30, D31, D32, D33, D34, D35, D36, D37, D38, D39, D4, D40, D41, D42, D43, D44, D45, D46, D47, D48, D49, D5, D50, D51, D52, D53, D54, D55, D56, D57, D58, D59, D6, D60, D61, D62, D63, D64, D65, D66, D67, D68, D69, D7, D70, D71, D72, D73, D74, D75, D76, D77, D78, D79, D8, D9: D_Small, Diode_SMD:D_SOD-123, symbol Device:D_Small
- added J1: TFT225P, Connector_PinHeader_2.54mm:PinHeader_1x08_P2.54mm_Vertical, symbol Connector:Conn_01x08_Pin
- added R1, R11, R12: 5.1k, Resistor_SMD:R_0805_2012Metric_Pad1.20x1.40mm_HandSolder, symbol Device:R_Small
- added U1: RotaryEncoder_Switch, Rotary_Encoder:RotaryEncoder_Bourns_Horizontal_PEC09-2xxxF-Sxxxx, symbol Device:RotaryEncoder_Switch
- added U10, U11, U12, U13, U14, U15, U16, U17, U18, U19, U2, U20, U21, U22, U23, U24, U25, U26, U27, U28, U3, U31, U32, U33, U34, U35, U36, U37, U38, U39, U4, U40, U41, U42, U45, U46, U47, U48, U49, U5, U50, U51, U52, U53, U54, U55, U58, U59, U6, U60, U61, U62, U63, U64, U65, U66, U67, U69, U7, U70, U76, U77, U78, U79, U8, U9: CherryMX_LTST-A683CEGBW, CherryMX_PCB_KailhSocket_LTST-A683CEGBW-HS:CherryMX_1.00u_PCB_KailhSocket_LTST-A683CEGBW-HS, symbol CherryMX:CherryMX_LTST-A683CEGBW
- added U29: CherryMX_LTST-A683CEGBW, CherryMX_PCB_KailhSocket_LTST-A683CEGBW-HS:CherryMX_2.00u_PCB_KailhSocket_LTST-A683CEGBW-HS, symbol CherryMX:CherryMX_LTST-A683CEGBW
- added U30, U43, U71, U73: CherryMX_LTST-A683CEGBW, CherryMX_PCB_KailhSocket_LTST-A683CEGBW-HS:CherryMX_1.50u_PCB_KailhSocket_LTST-A683CEGBW-HS, symbol CherryMX:CherryMX_LTST-A683CEGBW
- added U44, U68: CherryMX_LTST-A683CEGBW, CherryMX_PCB_KailhSocket_LTST-A683CEGBW-HS:CherryMX_1.75u_PCB_KailhSocket_LTST-A683CEGBW-HS, symbol CherryMX:CherryMX_LTST-A683CEGBW
- added U56, U57: CherryMX_LTST-A683CEGBW, CherryMX_PCB_KailhSocket_LTST-A683CEGBW-HS:CherryMX_2.25u_PCB_KailhSocket_LTST-A683CEGBW-HS, symbol CherryMX:CherryMX_LTST-A683CEGBW
- added U72, U75: CherryMX_LTST-A683CEGBW, CherryMX_PCB_KailhSocket_LTST-A683CEGBW-HS:CherryMX_1.25u_PCB_KailhSocket_LTST-A683CEGBW-HS, symbol CherryMX:CherryMX_LTST-A683CEGBW
- added U74: CherryMX_LTST-A683CEGBW, CherryMX_PCB_KailhSocket_LTST-A683CEGBW-HS:CherryMX_6.50u_PCB_KailhSocket_LTST-A683CEGBW-HS, symbol CherryMX:CherryMX_LTST-A683CEGBW
- BOOT1: renamed from SW2; footprint (none) -> Button_Switch_SMD:SW_SPST_TL3342
- C80: renamed from C3; footprint (none) -> Capacitor_SMD:C_0805_2012Metric_Pad1.18x1.45mm_HandSolder
- C81: renamed from C4; footprint (none) -> Capacitor_SMD:C_0805_2012Metric_Pad1.18x1.45mm_HandSolder
- C82: renamed from C?; footprint (none) -> Capacitor_SMD:C_0805_2012Metric_Pad1.18x1.45mm_HandSolder
- C83: renamed from C5; footprint (none) -> Capacitor_SMD:C_0805_2012Metric_Pad1.18x1.45mm_HandSolder
- C84: renamed from C6; footprint (none) -> Capacitor_SMD:C_0805_2012Metric_Pad1.18x1.45mm_HandSolder
- C85: renamed from C7; footprint (none) -> Capacitor_SMD:C_0805_2012Metric_Pad1.18x1.45mm_HandSolder
- C86: renamed from C8; footprint (none) -> Capacitor_SMD:C_0805_2012Metric_Pad1.18x1.45mm_HandSolder
- C87: renamed from C2; footprint (none) -> Capacitor_SMD:C_0805_2012Metric_Pad1.18x1.45mm_HandSolder
- C88: renamed from C9; footprint (none) -> Capacitor_SMD:C_0805_2012Metric_Pad1.18x1.45mm_HandSolder
- C89: renamed from C10; footprint (none) -> Capacitor_SMD:C_0805_2012Metric_Pad1.18x1.45mm_HandSolder
- C90: renamed from C1; footprint (none) -> Capacitor_SMD:C_0805_2012Metric_Pad1.18x1.45mm_HandSolder
- C91: renamed from C11; footprint (none) -> Capacitor_SMD:C_0805_2012Metric_Pad1.18x1.45mm_HandSolder
- F1: footprint (none) -> Fuse:Fuse_0805_2012Metric_Pad1.15x1.40mm_HandSolder
- J2: renamed from J1; footprint (none) -> Connector_USB:USB_C_Receptacle_HRO_TYPE-C-31-M-12
- J3: footprint (none) -> Connector_PinHeader_2.54mm:PinHeader_1x05_P2.54mm_Vertical
- J4: renamed from J2; footprint (none) -> Connector_JST:JST_SH_SM04B-SRSS-TB_1x04-1MP_P1.00mm_Horizontal
- R10, R2, R8: renamed from R?; footprint (none) -> Resistor_SMD:R_0805_2012Metric_Pad1.20x1.40mm_HandSolder
- R3: renamed from R1; footprint (none) -> Resistor_SMD:R_0805_2012Metric_Pad1.20x1.40mm_HandSolder
- R4: footprint (none) -> Resistor_SMD:R_0805_2012Metric_Pad1.20x1.40mm_HandSolder
- R5: renamed from R6; footprint (none) -> Resistor_SMD:R_0805_2012Metric_Pad1.20x1.40mm_HandSolder
- R6: renamed from R5; footprint (none) -> Resistor_SMD:R_0805_2012Metric_Pad1.20x1.40mm_HandSolder
- R7: renamed from R2; footprint (none) -> Resistor_SMD:R_0805_2012Metric_Pad1.20x1.40mm_HandSolder
- R9: renamed from R3; footprint (none) -> Resistor_SMD:R_0805_2012Metric_Pad1.20x1.40mm_HandSolder
- RST1: renamed from SW1; footprint (none) -> Button_Switch_SMD:SW_SPST_TL3342
- Y1: footprint (none) -> Crystal:Crystal_SMD_3225-4Pin_3.2x2.5mm_HandSoldering
- renumbered U1 to U80, U4 to U81, U2 to U82, U3 to U83
Connections:
- net +1V1: now also C92.1; no longer BOOT1.1, C80.2, C81.2, C82.2, C83.2, C84.2, C85.2, C86.2, C87.2, C88.1, C89.1, C90.2, C91.2, J2.A1 (GND), J2.A12 (GND), J2.B1 (GND), J2.B12 (GND), J2.S1 (SHIELD), J3.3 (Pin_3), J4.4 (Pin_4), R2.2, R3.2, RST1.1, U80.19 (TESTEN), U80.57 (GND), U81.2 (VN), U82.1 (GND), U83.4 (GND), Y1.2, Y1.4
- net +3V3: now also C1.1, C10.1, C11.1, C12.1, C13.1, C14.1, C15.1, C16.1, C17.1, C18.1, C19.1, C2.1, C20.1, C21.1, C22.1, C23.1, C24.1, C25.1, C26.1, C27.1, C28.1, C29.1, C3.1, C30.1, C31.1, C32.1, C33.1, C34.1, C35.1, C36.1, C37.1, C38.1, C39.1, C4.1, C40.1, C41.1, C42.1, C43.1, C44.1, C45.1, C46.1, C47.1, C48.1, C49.1, C5.1, C50.1, C51.1, C52.1, C53.1, C54.1, C55.1, C56.1, C57.1, C58.1, C59.1, C6.1, C60.1, C61.1, C62.1, C63.1, C64.1, C65.1, C66.1, C67.1, C68.1, C69.1, C7.1, C70.1, C71.1, C72.1, C73.1, C74.1, C75.1, C76.1, C77.1, C78.1, C79.1, C8.1, C9.1, C93.1, C94.1, C95.1, J1.2 (Pin_2), R1.1, R11.1, R12.1, U10.6 (VDD), U11.6 (VDD), U12.6 (VDD), U13.6 (VDD), U14.6 (VDD), U15.6 (VDD), U16.6 (VDD), U17.6 (VDD), U18.6 (VDD), U19.6 (VDD), U2.6 (VDD), U20.6 (VDD), U21.6 (VDD), U22.6 (VDD), U23.6 (VDD), U24.6 (VDD), U25.6 (VDD), U26.6 (VDD), U27.6 (VDD), U28.6 (VDD), U29.6 (VDD), U3.6 (VDD), U30.6 (VDD), U31.6 (VDD), U32.6 (VDD), U33.6 (VDD), U34.6 (VDD), U35.6 (VDD), U36.6 (VDD), U37.6 (VDD), U38.6 (VDD), U39.6 (VDD), U4.6 (VDD), U40.6 (VDD), U41.6 (VDD), U42.6 (VDD), U43.6 (VDD), U44.6 (VDD), U45.6 (VDD), U46.6 (VDD), U47.6 (VDD), U48.6 (VDD), U49.6 (VDD), U5.6 (VDD), U50.6 (VDD), U51.6 (VDD), U52.6 (VDD), U53.6 (VDD), U54.6 (VDD), U55.6 (VDD), U56.6 (VDD), U57.6 (VDD), U58.6 (VDD), U59.6 (VDD), U6.6 (VDD), U60.6 (VDD), U61.6 (VDD), U62.6 (VDD), U63.6 (VDD), U64.6 (VDD), U65.6 (VDD), U66.6 (VDD), U67.6 (VDD), U68.6 (VDD), U69.6 (VDD), U7.6 (VDD), U70.6 (VDD), U71.6 (VDD), U72.6 (VDD), U73.6 (VDD), U74.6 (VDD), U75.6 (VDD), U76.6 (VDD), U77.6 (VDD), U78.6 (VDD), U79.6 (VDD), U8.6 (VDD), U9.6 (VDD)
- net +5V: now also J4.4 (Pin_4); no longer J4.1 (Pin_1)
- net Col9: now reaches U80.11 (GPIO8)
- net Col9: now also U10.2, U25.2, U39.2, U53.2, U66.2
- net Col10: now reaches U80.12 (GPIO9)
- net Col10: now also U11.2, U26.2, U40.2, U54.2, U67.2, U75.2
- net Col11: now reaches U80.13 (GPIO10)
- net Col11: now also U12.2, U27.2, U41.2, U55.2, U68.2, U76.2
- net Col12: now reaches U80.14 (GPIO11)
- net Col12: now also U13.2, U28.2, U42.2, U56.2, U77.2
- net Col13: now reaches U80.15 (GPIO12)
- net Col13: now also U14.2, U29.2, U43.2, U69.2, U78.2
- net Col14: now reaches U80.16 (GPIO13)
- net Col14: now also U15.2, U70.2, U79.2
- net Row0: now reaches U80.17 (GPIO14)
- net Row0: now also D1.1 (K), D10.1 (K), D11.1 (K), D12.1 (K), D13.1 (K), D14.1 (K), D15.1 (K), D2.1 (K), D3.1 (K), D4.1 (K), D5.1 (K), D6.1 (K), D7.1 (K), D8.1 (K), D9.1 (K)
- net Row1: now reaches U80.18 (GPIO15)
- net Row1: now also D16.1 (K), D17.1 (K), D18.1 (K), D19.1 (K), D20.1 (K), D21.1 (K), D22.1 (K), D23.1 (K), D24.1 (K), D25.1 (K), D26.1 (K), D27.1 (K), D28.1 (K), D29.1 (K)
- net Col0: now reaches U80.2 (GPIO0)
- net Col0: now also U1.S1, U16.2, U30.2, U44.2, U57.2, U71.2
- net Row2: now reaches U80.27 (GPIO16)
- net Row2: now also D30.1 (K), D31.1 (K), D32.1 (K), D33.1 (K), D34.1 (K), D35.1 (K), D36.1 (K), D37.1 (K), D38.1 (K), D39.1 (K), D40.1 (K), D41.1 (K), D42.1 (K), D43.1 (K)
- net Row3: now reaches U80.28 (GPIO17)
- net Row3: now also D44.1 (K), D45.1 (K), D46.1 (K), D47.1 (K), D48.1 (K), D49.1 (K), D50.1 (K), D51.1 (K), D52.1 (K), D53.1 (K), D54.1 (K), D55.1 (K), D56.1 (K)
- net SCL: now reaches U80.29 (GPIO18)
- net SCL: now also J1.3 (Pin_3)
- net Col1: now reaches U80.3 (GPIO1)
- net Col1: now also U17.2, U2.2, U31.2, U45.2, U58.2, U72.2
- net SDA: now reaches U80.30 (GPIO19)
- net SDA: now also J1.4 (Pin_4)
- net RES: now reaches U80.31 (GPIO20)
- net RES: now also J1.5 (Pin_5), R1.2
- net DC: now reaches U80.32 (GPIO21)
- net DC: now also J1.6 (Pin_6)
- net Row4: now reaches U80.34 (GPIO22)
- net Row4: now also D57.1 (K), D58.1 (K), D59.1 (K), D60.1 (K), D61.1 (K), D62.1 (K), D63.1 (K), D64.1 (K), D65.1 (K), D66.1 (K), D67.1 (K), D68.1 (K), D69.1 (K), D70.1 (K)
- net Row5: now reaches U80.35 (GPIO23)
- net Row5: now also D71.1 (K), D72.1 (K), D73.1 (K), D74.1 (K), D75.1 (K), D76.1 (K), D77.1 (K), D78.1 (K), D79.1 (K)
- net Arot: now reaches U80.36 (GPIO24)
- net Arot: now also R12.2, U1.A
- net Brot: now reaches U80.37 (GPIO25)
- net Brot: now also R11.2, U1.B
- net CS: now reaches U80.38 (GPIO26_ADC0)
- net CS: now also J1.7 (Pin_7)
- net BLK: now reaches U80.39 (GPIO27_ADC1)
- net BLK: now also J1.8 (Pin_8)
- net Col3: now reaches U80.4 (GPIO2)
- net Col3: now also U19.2, U33.2, U4.2, U47.2, U60.2
- net RGB_Data1: now reaches U80.41 (GPIO29_ADC3)
- net RGB_Data1: now also U2.4 (DIN)
- net Col4: now reaches U80.5 (GPIO3)
- net Col4: now also U20.2, U34.2, U48.2, U5.2, U61.2
- net Col5: now reaches U80.6 (GPIO4)
- net Col5: now also U21.2, U35.2, U49.2, U6.2, U62.2
- net Col6: now reaches U80.7 (GPIO5)
- net Col7: now reaches U80.8 (GPIO6)
- net Col7: now also U23.2, U37.2, U51.2, U64.2, U74.2, U8.2
- net Col8: now reaches U80.9 (GPIO7)
- net Col8: now also U24.2, U38.2, U52.2, U65.2, U9.2
- new net: D77.2 (A), U77.1
- new net: U76.5 (DOUT), U77.4 (DIN)
- new net: U77.5 (DOUT), U78.4 (DIN)
- new net: D64.2 (A), U64.1
- new net: D73.2 (A), U73.1
- new net: U72.5 (DOUT), U73.4 (DIN)
- new net: U73.5 (DOUT), U74.4 (DIN)
- new net: D71.2 (A), U71.1
- new net: D34.2 (A), U34.1
- new net: D58.2 (A), U58.1
- new net: U57.5 (DOUT), U58.4 (DIN)
- new net: U58.5 (DOUT), U59.4 (DIN)
- new net: D21.2 (A), U21.1
- new net: U20.5 (DOUT), U21.4 (DIN)
- new net: U21.5 (DOUT), U22.4 (DIN)
- new net: D65.2 (A), U65.1
- new net: D14.2 (A), U14.1
- new net: D23.2 (A), U23.1
- new net: D24.2 (A), U24.1
- new net: D31.2 (A), U31.1
- new net: D67.2 (A), U67.1
- new net: D1.2 (A), U1.S2
- new net: D55.2 (A), U55.1
- new net: D5.2 (A), U5.1
- new net: D38.2 (A), U38.1
- new net: U37.5 (DOUT), U38.4 (DIN)
- new net: U38.5 (DOUT), U39.4 (DIN)
- new net: D2.2 (A), U2.1
- new net: U2.5 (DOUT), U3.4 (DIN)
- new net: D70.2 (A), U70.1
- new net: D61.2 (A), U61.1
- new net: D46.2 (A), U46.1
- new net: D7.2 (A), U7.1
- new net: D18.2 (A), U18.1
- new net: U17.5 (DOUT), U18.4 (DIN)
- new net: U18.5 (DOUT), U19.4 (DIN)
- new net: D72.2 (A), U72.1
- new net: D10.2 (A), U10.1
- new net: U10.4 (DIN), U9.5 (DOUT)
- new net: U10.5 (DOUT), U11.4 (DIN)
- new net: D49.2 (A), U49.1
- new net: U48.5 (DOUT), U49.4 (DIN)
- new net: U49.5 (DOUT), U50.4 (DIN)
- new net: D40.2 (A), U40.1
- new net: U39.5 (DOUT), U40.4 (DIN)
- new net: U40.5 (DOUT), U41.4 (DIN)
- new net: D48.2 (A), U48.1
- new net: U47.5 (DOUT), U48.4 (DIN)
- new net: D6.2 (A), U6.1
- new net: D37.2 (A), U37.1
- new net: D56.2 (A), U56.1
- new net: D63.2 (A), U63.1
- new net: U22.2, U36.2, U50.2, U63.2, U7.2
- new net: U62.5 (DOUT), U63.4 (DIN)
- new net: U63.5 (DOUT), U64.4 (DIN)
- new net: U22.5 (DOUT), U23.4 (DIN)
- new net: U23.5 (DOUT), U24.4 (DIN)
- new net: D44.2 (A), U44.1
- new net: U44.5 (DOUT), U45.4 (DIN)
- new net: D36.2 (A), U36.1
- new net: D52.2 (A), U52.1
- new net: U51.5 (DOUT), U52.4 (DIN)
- new net: U52.5 (DOUT), U53.4 (DIN)
- new net: D12.2 (A), U12.1
- new net: U11.5 (DOUT), U12.4 (DIN)
- new net: U12.5 (DOUT), U13.4 (DIN)
- new net: D16.2 (A), U16.1
- new net: D4.2 (A), U4.1
- new net: U3.5 (DOUT), U4.4 (DIN)
- new net: U4.5 (DOUT), U5.4 (DIN)
- new net: D79.2 (A), U79.1
- new net: D22.2 (A), U22.1
- new net: U6.5 (DOUT), U7.4 (DIN)
- new net: U7.5 (DOUT), U8.4 (DIN)
- new net: D19.2 (A), U19.1
- new net: U19.5 (DOUT), U20.4 (DIN)
- new net: D9.2 (A), U9.1
- new net: D57.2 (A), U57.1
- new net: D62.2 (A), U62.1
- new net: U33.5 (DOUT), U34.4 (DIN)
- new net: U34.5 (DOUT), U35.4 (DIN)
- new net: U8.5 (DOUT), U9.4 (DIN)
- new net: U24.5 (DOUT), U25.4 (DIN)
- new net: D29.2 (A), U29.1
- new net: D78.2 (A), U78.1
- new net: D66.2 (A), U66.1
- new net: U65.5 (DOUT), U66.4 (DIN)
- new net: U66.5 (DOUT), U67.4 (DIN)
- new net: D69.2 (A), U69.1
- new net: U68.5 (DOUT), U69.4 (DIN)
- new net: U69.5 (DOUT), U70.4 (DIN)
- new net: D35.2 (A), U35.1
- new net: U35.5 (DOUT), U36.4 (DIN)
- new net: D20.2 (A), U20.1
- new net: U71.5 (DOUT), U72.4 (DIN)
- new net: D41.2 (A), U41.1
- new net: U41.5 (DOUT), U42.4 (DIN)
- new net: D59.2 (A), U59.1
- new net: U30.5 (DOUT), U31.4 (DIN)
- new net: U31.5 (DOUT), U32.4 (DIN)
- new net: D11.2 (A), U11.1
- new net: D51.2 (A), U51.1
- new net: D28.2 (A), U28.1
- new net: D45.2 (A), U45.1
- new net: U45.5 (DOUT), U46.4 (DIN)
- new net: D42.2 (A), U42.1
- new net: D26.2 (A), U26.1
- new net: D27.2 (A), U27.1
- new net: D39.2 (A), U39.1
- new net: D32.2 (A), U32.1
- new net: D43.2 (A), U43.1
- new net: U42.5 (DOUT), U43.4 (DIN)
- new net: D30.2 (A), U30.1
- new net: U67.5 (DOUT), U68.4 (DIN)
- new net: D25.2 (A), U25.1
- new net: U25.5 (DOUT), U26.4 (DIN)
- new net: U26.5 (DOUT), U27.4 (DIN)
- new net: D50.2 (A), U50.1
- new net: U36.5 (DOUT), U37.4 (DIN)
- new net: D33.2 (A), U33.1
- new net: U32.5 (DOUT), U33.4 (DIN)
- new net: U28.5 (DOUT), U29.4 (DIN)
- new net: U13.5 (DOUT), U14.4 (DIN)
- new net: U14.5 (DOUT), U15.4 (DIN)
- new net: D3.2 (A), U3.1
- new net: U60.5 (DOUT), U61.4 (DIN)
- new net: U61.5 (DOUT), U62.4 (DIN)
- new net: U55.5 (DOUT), U56.4 (DIN)
- new net: U50.5 (DOUT), U51.4 (DIN)
- new net: U54.5 (DOUT), U55.4 (DIN)
- new net: U78.5 (DOUT), U79.4 (DIN)
- new net: U16.5 (DOUT), U17.4 (DIN)
- new net: D76.2 (A), U76.1
- new net: U75.5 (DOUT), U76.4 (DIN)
- new net: D74.2 (A), U74.1
- new net: D54.2 (A), U54.1
- new net: U53.5 (DOUT), U54.4 (DIN)
- new net: U59.5 (DOUT), U60.4 (DIN)
- new net: U64.5 (DOUT), U65.4 (DIN)
- new net: D60.2 (A), U60.1
- new net: D53.2 (A), U53.1
- new net: D15.2 (A), U15.1
- new net: D47.2 (A), U47.1
- new net: U46.5 (DOUT), U47.4 (DIN)
- new net: U5.5 (DOUT), U6.4 (DIN)
- new net: D8.2 (A), U8.1
- new net: D13.2 (A), U13.1
- new net: D68.2 (A), U68.1
- new net: D17.2 (A), U17.1
- new net: U74.5 (DOUT), U75.4 (DIN)
- new net: D75.2 (A), U75.1
- new net: U27.5 (DOUT), U28.4 (DIN)
- new net Col2: U18.2, U3.2, U32.2, U46.2, U59.2, U73.2
- new net GND: BOOT1.1, C1.2, C10.2, C11.2, C12.2, C13.2, C14.2, C15.2, C16.2, C17.2, C18.2, C19.2, C2.2, C20.2, C21.2, C22.2, C23.2, C24.2, C25.2, C26.2, C27.2, C28.2, C29.2, C3.2, C30.2, C31.2, C32.2, C33.2, C34.2, C35.2, C36.2, C37.2, C38.2, C39.2, C4.2, C40.2, C41.2, C42.2, C43.2, C44.2, C45.2, C46.2, C47.2, C48.2, C49.2, C5.2, C50.2, C51.2, C52.2, C53.2, C54.2, C55.2, C56.2, C57.2, C58.2, C59.2, C6.2, C60.2, C61.2, C62.2, C63.2, C64.2, C65.2, C66.2, C67.2, C68.2, C69.2, C7.2, C70.2, C71.2, C72.2, C73.2, C74.2, C75.2, C76.2, C77.2, C78.2, C79.2, C8.2, C80.2, C81.2, C82.2, C83.2, C84.2, C85.2, C86.2, C87.2, C88.1, C89.1, C9.2, C90.2, C91.2, C92.2, C93.2, C94.2, C95.2, J1.1 (Pin_1), J2.A1 (GND), J2.A12 (GND), J2.B1 (GND), J2.B12 (GND), J2.S1 (SHIELD), J3.3 (Pin_3), J4.1 (Pin_1), R2.2, R3.2, RST1.1, U1.C, U10.3 (VSS), U11.3 (VSS), U12.3 (VSS), U13.3 (VSS), U14.3 (VSS), U15.3 (VSS), U16.3 (VSS), U17.3 (VSS), U18.3 (VSS), U19.3 (VSS), U2.3 (VSS), U20.3 (VSS), U21.3 (VSS), U22.3 (VSS), U23.3 (VSS), U24.3 (VSS), U25.3 (VSS), U26.3 (VSS), U27.3 (VSS), U28.3 (VSS), U29.3 (VSS), U3.3 (VSS), U30.3 (VSS), U31.3 (VSS), U32.3 (VSS), U33.3 (VSS), U34.3 (VSS), U35.3 (VSS), U36.3 (VSS), U37.3 (VSS), U38.3 (VSS), U39.3 (VSS), U4.3 (VSS), U40.3 (VSS), U41.3 (VSS), U42.3 (VSS), U43.3 (VSS), U44.3 (VSS), U45.3 (VSS), U46.3 (VSS), U47.3 (VSS), U48.3 (VSS), U49.3 (VSS), U5.3 (VSS), U50.3 (VSS), U51.3 (VSS), U52.3 (VSS), U53.3 (VSS), U54.3 (VSS), U55.3 (VSS), U56.3 (VSS), U57.3 (VSS), U58.3 (VSS), U59.3 (VSS), U6.3 (VSS), U60.3 (VSS), U61.3 (VSS), U62.3 (VSS), U63.3 (VSS), U64.3 (VSS), U65.3 (VSS), U66.3 (VSS), U67.3 (VSS), U68.3 (VSS), U69.3 (VSS), U7.3 (VSS), U70.3 (VSS), U71.3 (VSS), U72.3 (VSS), U73.3 (VSS), U74.3 (VSS), U75.3 (VSS), U76.3 (VSS), U77.3 (VSS), U78.3 (VSS), U79.3 (VSS), U8.3 (VSS), U80.19 (TESTEN), U80.57 (GND), U81.2 (VN), U82.1 (GND), U83.4 (GND), U9.3 (VSS), Y1.2, Y1.4
- new net RGB_DATA2: U15.5 (DOUT), U16.4 (DIN)
- new net RGB_DATA3: U30.4 (DIN)
- new net RGB_DATA4: U43.5 (DOUT), U44.4 (DIN)
- new net RGB_DATA5: U56.5 (DOUT), U57.4 (DIN)
- new net RGB_DATA6: U70.5 (DOUT), U71.4 (DIN)
- no-connect marks 4 -> 6
Other:
- note added: "CRYSTAL"
- note added: "DECOUPLING"
- note added: "FLASH"
- note added: "RESET"
- note added: "RP2040"
- note added: "TFT2.25"
- note added: "USB_C"
- note added: "V. REGULATOR"
- moved on the sheet: BOOT1, C80, C81, C82, C83, C84, C85, C86, C87, C88, C89, C90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

Commit message: update to rp20 keyboard pcb
Parts:
- removed C1: 100n, Capacitor_SMD:C_0805_2012Metric_Pad1.18x1.45mm_HandSolder, symbol Device:C_Small
- added S1: MX_stab, PCM_marbastlib-mx:STAB_MX_P_2u, symbol PCM_marbastlib-mx:MX_stab
- added S3: MX_stab, PCM_marbastlib-mx:STAB_MX_P_2.25u, symbol PCM_marbastlib-mx:MX_stab
- added S5: MX_stab, PCM_marbastlib-mx:STAB_MX_2.25u, symbol PCM_marbastlib-mx:MX_stab
- added S6: MX_stab, PCM_marbastlib-mx:STAB_MX_P_7u, symbol PCM_marbastlib-mx:MX_stab
- renumbered D2 to D1, D11 to D10, D12 to D11, D13 to D12, D14 to D13, D15 to D14, D16 to D15, D17 to D16, D18 to D17, D19 to D18, D20 to D19, D3 to D2, D21 to D20, D22 to D21, D23 to D22, D24 to D23, D25 to D24, D26 to D25, D27 to D26, D28 to D27, D29 to D28, D30 to D29, D4 to D3, D31 to D30, D32 to D31, D33 to D32, D34 to D33, D35 to D34, D36 to D35, D37 to D36, D38 to D37, D39 to D38, D40 to D39, D5 to D4, D41 to D40, D42 to D41, D43 to D42, D44 to D43, D45 to D44, D46 to D45, D47 to D46, D48 to D47, D49 to D48, D50 to D49, D6 to D5, D51 to D50, D52 to D51, D53 to D52, D54 to D53, D55 to D54, D56 to D55, D57 to D56, D58 to D57, D59 to D58, D60 to D59, D7 to D6, D61 to D60, D62 to D61, D63 to D62, D64 to D63, D65 to D64, D66 to D65, D67 to D66, D68 to D67, D69 to D68, D70 to D69, D8 to D7, D71 to D70, D72 to D71, D73 to D72, D74 to D73, D75 to D74, D76 to D75, D77 to D76, D78 to D77, D79 to D78, D1 to D79, D9 to D8, D10 to D9, U2 to U1, U11 to U10, U12 to U11, U13 to U12, U14 to U13, U15 to U14, U16 to U15, U17 to U16, U18 to U17, U19 to U18, U20 to U19, U3 to U2, U21 to U20, U22 to U21, U23 to U22, U24 to U23, U25 to U24, U26 to U25, U27 to U26, U28 to U27, U29 to U28, U30 to U29, U4 to U3, U31 to U30, U32 to U31, U33 to U32, U34 to U33, U35 to U34, U36 to U35, U37 to U36, U38 to U37, U39 to U38, U40 to U39, U5 to U4, U41 to U40, U42 to U41, U43 to U42, U44 to U43, U45 to U44, U46 to U45, U47 to U46, U48 to U47, U49 to U48, U50 to U49, U6 to U5, U51 to U50, U52 to U51, U53 to U52, U54 to U53, U55 to U54, U56 to U55, U57 to U56, U58 to U57, U59 to U58, U60 to U59, U7 to U6, U61 to U60, U62 to U61, U63 to U62, U64 to U63, U65 to U64, U66 to U65, U67 to U66, U68 to U67, U69 to U68, U70 to U69, U8 to U7, U71 to U70, U72 to U71, U73 to U72, U74 to U73, U75 to U74, U76 to U75, U77 to U76, U78 to U77, U79 to U78, U1 to U79, U9 to U8, U10 to U9
Connections:
- net +3V3: now also J3.4 (Pin_4); no longer J3.2 (Pin_2)
- net Arot: now also U80.38 (GPIO26_ADC0); no longer U80.36 (GPIO24)
- net BLK: now also U80.37 (GPIO25); no longer U80.39 (GPIO27_ADC1)
- net Brot: now also U80.39 (GPIO27_ADC1); no longer U80.37 (GPIO25)
- net CS: now also U80.36 (GPIO24); no longer U80.38 (GPIO26_ADC0)
- net Col10: now also U80.13 (GPIO10); no longer U80.12 (GPIO9)
- net Col11: now also U80.14 (GPIO11); no longer U80.13 (GPIO10)
- net Col12: now also U80.15 (GPIO12); no longer U80.14 (GPIO11)
- net Col13: now also U80.16 (GPIO13); no longer U80.15 (GPIO12)
- net Col14: now also U80.32 (GPIO21); no longer U80.16 (GPIO13)
- net Col2: now also U80.4 (GPIO2)
- net Col3: now also U80.5 (GPIO3); no longer U80.4 (GPIO2)
- net Col4: now also U80.6 (GPIO4); no longer U80.5 (GPIO3)
- net Col5: now also U80.7 (GPIO5); no longer U80.6 (GPIO4)
- net Col6: now also U21.2, U35.2, U49.2, U6.2, U62.2, U80.8 (GPIO6); no longer U80.7 (GPIO5)
- net Col7: now also U80.9 (GPIO7); no longer U80.8 (GPIO6)
- net Col8: now also U80.11 (GPIO8); no longer U80.9 (GPIO7)
- net Col9: now also U80.12 (GPIO9); no longer U80.11 (GPIO8)
- net DC: now also U80.35 (GPIO23); no longer U80.32 (GPIO21)
- net GND: now also J3.5 (Pin_5); no longer J3.3 (Pin_3)
- net RES: now also U80.34 (GPIO22); no longer U80.31 (GPIO20)
- net RGB_DATA3: now also U28.5 (DOUT)
- net Row0: now also U80.40 (GPIO28_ADC2); no longer U80.17 (GPIO14)
- net Row2: now also U80.17 (GPIO14); no longer U80.27 (GPIO16)
- net Row3: now also U80.31 (GPIO20); no longer U80.28 (GPIO17)
- net Row4: now also U80.27 (GPIO16); no longer U80.34 (GPIO22)
- net Row5: now also U80.28 (GPIO17); no longer U80.35 (GPIO23)
- net SWC: now also J3.2 (Pin_2); no longer J3.4 (Pin_4)
- net SWD: now also J3.3 (Pin_3); no longer J3.5 (Pin_5)
- no-connect marks 6 -> 5
